Commit message: fix: 更新aubo_description仓库

File: urdf/aubo_C5.urdf (robot description, URDF)
Before this commit: robot aubo_C5, 8 links, 7 joints
Joints:
- joint foreArm_joint: limit lower=-6.283185307179586476925286766559 upper=6.283185307179586476925286766559 effort=133 velocity=2.5964 -> lower=-6.283185307179586476925286766559 upper=6.283185307179586476925286766559 effort=133 velocity=2.565634
- joint shoulder_joint: limit lower=-6.283185307179586476925286766559 upper=6.283185307179586476925286766559 effort=133 velocity=2.5964 -> lower=-6.283185307179586476925286766559 upper=6.283185307179586476925286766559 effort=133 velocity=2.565634
- joint upperArm_joint: limit lower=-6.283185307179586476925286766559 upper=6.283185307179586476925286766559 effort=133 velocity=2.5964 -> lower=-6.283185307179586476925286766559 upper=6.283185307179586476925286766559 effort=133 velocity=2.565634
- joint wrist1_joint: limit lower=-6.283185307179586476925286766559 upper=6.283185307179586476925286766559 effort=13.5 velocity=3.1105 -> lower=-6.283185307179586476925286766559 upper=6.283185307179586476925286766559 effort=13.5 velocity=3.106686
- joint wrist2_joint: limit lower=-6.283185307179586476925286766559 upper=6.283185307179586476925286766559 effort=13.5 velocity=3.1105 -> lower=-6.283185307179586476925286766559 upper=6.283185307179586476925286766559 effort=13.5 velocity=3.106686
- joint wrist3_joint: limit lower=-6.283185307179586476925286766559 upper=6.283185307179586476925286766559 effort=13.5 velocity=3.1105 -> lower=-6.283185307179586476925286766559 upper=6.283185307179586476925286766559 effort=13.5 velocity=3.106686

File: urdf/aubo_E10_10.urdf (robot description, URDF)
Before this commit: robot aubo_E10_10, 8 links, 7 joints
Links:
- link base_link: mass 1.2345 -> 2.592000
- link foreArm_Link: mass 3.1022 -> 4.448092
- link shoulder_Link: mass 10.994 -> 10.180139
- link upperArm_Link: mass 5.3139 -> 18.096361
- link wrist1_Link: mass 0.57981 -> 1.791660
- link wrist2_Link: mass 0.57981 -> 1.791660
- link wrist3_Link: mass 0.13669 -> 0.197800

File: urdf/aubo_E3.urdf (robot description, URDF)
Before this commit: robot aubo_E3, 8 links, 7 joints
Links:
- link base_link: mass 0.97332 -> 1.365846
- link foreArm_Link: mass 1.5214 -> 2.351523
- link shoulder_Link: mass 1.173 -> 3.257300
- link upperArm_Link: mass 2.7791 -> 6.116851
- link wrist1_Link: mass 0.63348 -> 1.628022
- link wrist2_Link: mass 0.63348 -> 1.628022
- link wrist3_Link: mass 0.13713 -> 0.197800

File: urdf/aubo_E5_10.urdf (robot description, URDF)
Before this commit: robot aubo_E5_10, 8 links, 7 joints
Links:
- link base_link: mass 0.83419 -> 1.539020
- link foreArm_Link: mass 2.88 -> 2.849168
- link shoulder_Link: mass 5.05 -> 4.848581
- link upperArm_Link: mass 11.28 -> 10.836261
- link wrist1_Link: mass 1.62 -> 1.628022
- link wrist2_Link: mass 1.62 -> 1.628022
- link wrist3_Link: mass 0.5 -> 0.197800

File: urdf/aubo_LW2_1500.urdf (robot description, URDF)
Before this commit: robot aubo_LW2_1500, 8 links, 7 joints
Links:
- link base_link: mass 0.372514960613725 -> 2.0138283
- link foreArm_Link: mass 0.0692813683277528 -> 0.96538834
- link shoulder_Link: mass 0.328105939234581 -> 3.60778729; geometry collision mesh filename=package://aubo_description/meshes/aubo_LW2_1500/collision/l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; visual mesh filename=package://aubo_description/meshes/aubo_LW2_1500/visual/link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
- link upperArm_Link: mass 0.530501711854129 -> 2.30370284
- link wrist1_Link: mass 0.346296462439813 -> 1.5749858; geometry collision mesh filename=package://aubo_description/meshes/aubo_LW2_1500/collision/l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; visual mesh filename=package://aubo_description/meshes/aubo_LW2_1500/visual/link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
- link wrist2_Link: mass 0.0697044777353023 -> 0.96390764
- link wrist3_Link: mass 0.173734952383709 -> 0.20668692; geometry collision mesh filename=package://aubo_description/meshes/aubo_LW2_1500/collision/l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; visual mesh filename=package://aubo_description/meshes/aubo_LW2_1500/visual/link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
Joints:
- joint foreArm_joint: limit lower=-2.96705972839036 upper=2.96705972839036 effort=133 velocity=4.188790133 -> lower=-3.05432613888889 upper=3.05432613888889 effort=133 velocity=4.188790133; origin xyz=0.519 0 0.01764 rpy=3.1415926535897932384626433832795 0 -1.5707963267948966192313216916398 -> xyz=0.519 0 0.0176 rpy=3.1415926535897932384626433832795 0 -1.5707963267948966192313216916398
- joint shoulder_joint: limit lower=0 upper=4.71238898038469 effort=49 velocity=3.1415926535897932384626433832795 -> lower=-2.35619445 upper=2.35619445 effort=49 velocity=3.1415926535897932384626433832795; origin xyz=0 0 0.153 rpy=3.1415926535897932384626433832795 0 3.1415926535897932384626433832795 -> xyz=0 0 0.153 rpy=0 0 1.5707963267948966192313216916398
- joint upperArm_joint: origin xyz=0.208 0 0 rpy=1.5707963267948966192313216916398 0 0 -> xyz=-0.208 0 0 rpy=1.5707963267948966192313216916398 -1.5707963267948966192313216916398 0
- joint wrist2_joint: origin xyz=0 -0.09481 0 rpy=1.5707963267948966192313216916398 0 0 -> xyz=0 -0.09485 0 rpy=1.5707963267948966192313216916398 0 0

File: urdf/aubo_S3.urdf (robot description, URDF)
Before this commit: robot aubo_S3, 8 links, 7 joints
Joints:
- joint foreArm_joint: limit lower=-3.054326190990076759616458844855 upper=3.054326190990076759616458844855 effort=133 velocity=2.5964 -> lower=-2.87979326579064 upper=2.87979326579064 effort=39 velocity=2.5964; origin xyz=0.284 0 0 rpy=-3.1415926535897932384626433832795 0 0 -> xyz=0.2835 0 0 rpy=-3.1415926535897932384626433832795 0 0
- joint shoulder_joint: limit lower=-3.054326190990076759616458844855 upper=3.054326190990076759616458844855 effort=133 velocity=2.5964 -> lower=-6.283185307179586476925286766559 upper=6.283185307179586476925286766559 effort=49 velocity=2.5964
- joint upperArm_joint: limit lower=-3.054326190990076759616458844855 upper=3.054326190990076759616458844855 effort=133 velocity=2.5964 -> lower=-3.1415926535897932384626433832795 upper=3.1415926535897932384626433832795 effort=49 velocity=2.5964
- joint wrist1_joint: limit lower=-3.054326190990076759616458844855 upper=3.054326190990076759616458844855 effort=13.5 velocity=3.1105 -> lower=-6.283185307179586476925286766559 upper=6.283185307179586476925286766559 effort=9.8 velocity=3.1105
- joint wrist2_joint: limit lower=-3.054326190990076759616458844855 upper=3.054326190990076759616458844855 effort=13.5 velocity=3.1105 -> lower=-6.283185307179586476925286766559 upper=6.283185307179586476925286766559 effort=9.8 velocity=3.1105
- joint wrist3_joint: limit lower=-3.054326190990076759616458844855 upper=3.054326190990076759616458844855 effort=13.5 velocity=3.1105 -> lower=-6.283185307179586476925286766559 upper=6.283185307179586476925286766559 effort=9.8 velocity=3.1105

File: urdf/aubo_S5.urdf (robot description, URDF)
Before this commit: robot aubo_S5, 8 links, 7 joints
Links:
- link wrist2_Link: mass 1.06103669 -> 1.06823262
- link wrist3_Link: mass 0.22222939 -> 0.21445068
Joints:
- joint foreArm_joint: limit lower=-3.054326190990076759616458844855 upper=3.054326190990076759616458844855 effort=133 velocity=2.5964 -> lower=-2.87979326579064 upper=2.87979326579064 effort=49 velocity=2.5964
- joint shoulder_joint: limit lower=-3.054326190990076759616458844855 upper=3.054326190990076759616458844855 effort=133 velocity=2.5964 -> lower=-6.283185307179586476925286766559 upper=6.283185307179586476925286766559 effort=108 velocity=2.5964
- joint upperArm_joint: limit lower=-3.054326190990076759616458844855 upper=3.054326190990076759616458844855 effort=133 velocity=2.5964 -> lower=-3.1415926535897932384626433832795 upper=3.1415926535897932384626433832795 effort=108 velocity=2.5964
- joint wrist1_joint: limit lower=-3.054326190990076759616458844855 upper=3.054326190990076759616458844855 effort=13.5 velocity=3.1105 -> lower=-6.283185307179586476925286766559 upper=6.283185307179586476925286766559 effort=9.8 velocity=3.1105
- joint wrist2_joint: limit lower=-3.054326190990076759616458844855 upper=3.054326190990076759616458844855 effort=13.5 velocity=3.1105 -> lower=-6.283185307179586476925286766559 upper=6.283185307179586476925286766559 effort=9.8 velocity=3.1105; origin xyz=0 0.1305 0 rpy=-1.5707963267948966192313216916398 0 0 -> xyz=0 0.130 0 rpy=-1.5707963267948966192313216916398 0 0
- joint wrist3_joint: limit lower=-3.054326190990076759616458844855 upper=3.054326190990076759616458844855 effort=13.5 velocity=3.1105 -> lower=-6.283185307179586476925286766559 upper=6.283185307179586476925286766559 effort=9.8 velocity=3.1105; origin xyz=0 -0.1242 0 rpy=1.5707963267948966192313216916398 0 1.7907E-15 -> xyz=0 -0.1237 0 rpy=1.5707963267948966192313216916398 0 1.7907E-15

File: urdf/aubo_c5_30.urdf (robot description, URDF)
Before this commit: robot aubo_c5_30, 8 links, 7 joints
Links:
- link base_link: mass 0.83419 -> 1.539020
- link foreArm_Link: mass 2.88 -> 2.849168
- link shoulder_Link: mass 5.05 -> 4.848581
- link upperArm_Link: mass 11.28 -> 10.836261
- link wrist1_Link: mass 1.62 -> 1.6280228022
- link wrist2_Link: mass 1.62 -> 1.6280228022
- link wrist3_Link: mass 0.5 -> 0.197800

File: urdf/aubo_e10_10.urdf (robot description, URDF)
Before this commit: robot aubo_e10_10, 8 links, 7 joints
Links:
- link base_link: mass 1.2345 -> 2.592000
- link foreArm_Link: mass 3.1022 -> 4.448092
- link shoulder_Link: mass 10.994 -> 10.180139
- link upperArm_Link: mass 5.3139 -> 18.096361
- link wrist1_Link: mass 0.57981 -> 1.791660
- link wrist2_Link: mass 0.57981 -> 1.791660
- link wrist3_Link: mass 0.13669 -> 0.197800

File: urdf/aubo_i10_10.urdf (robot description, URDF)
Before this commit: robot aubo_i10_10, 8 links, 7 joints
Links:
- link base_link: mass 1.2345 -> 2.592000
- link foreArm_Link: mass 3.1022 -> 4.448092
- link shoulder_Link: mass 10.994 -> 10.180139
- link upperArm_Link: mass 5.3139 -> 18.096361
- link wrist1_Link: mass 0.57981 -> 1.791660
- link wrist2_Link: mass 0.57981 -> 1.791660
- link wrist3_Link: mass 0.13669 -> 0.197800

File: urdf/aubo_i10_11.urdf (robot description, URDF)
Before this commit: robot aubo_i10_11, 8 links, 7 joints
Links:
- link base_link: mass 1.2345 -> 2.592000
- link foreArm_Link: mass 3.1022 -> 4.448092
- link shoulder_Link: mass 10.994 -> 10.180139
- link upperArm_Link: mass 5.3139 -> 18.096361
- link wrist1_Link: mass 0.57981 -> 1.791660
- link wrist2_Link: mass 0.57981 -> 1.791660
- link wrist3_Link: mass 0.13669 -> 0.197800

File: urdf/aubo_i10_30.urdf (robot description, URDF)
Before this commit: robot aubo_i10_30, 8 links, 7 joints
Links:
- link base_link: mass 1.2345 -> 2.592000
- link foreArm_Link: mass 3.1022 -> 4.448092
- link shoulder_Link: mass 10.994 -> 10.180139
- link upperArm_Link: mass 5.3139 -> 18.096361
- link wrist1_Link: mass 0.57981 -> 1.791660
- link wrist2_Link: mass 0.57981 -> 1.791660
- link wrist3_Link: mass 0.13669 -> 0.197800

File: urdf/aubo_i12H.urdf (robot description, URDF)
Before this commit: robot aubo_i12H, 8 links, 7 joints
Links:
- link base_link: mass 1.0247 -> 2.592000
- link foreArm_Link: mass 4.3599 -> 4.393121
- link shoulder_Link: mass 11.1649 -> 10.180139
- link upperArm_Link: mass 19.3544 -> 18.169652
- link wrist1_Link: mass 2.5692 -> 2.370741
- link wrist2_Link: mass 2.5692 -> 2.370741
- link wrist3_Link: mass 0.203 -> 0.259654

File: urdf/aubo_i16H.urdf (robot description, URDF)
Before this commit: robot aubo_i16H, 8 links, 7 joints
Links:
- link base_link: mass 1.0247 -> 2.592000
- link foreArm_Link: mass 3.9474 -> 3.926354
- link shoulder_Link: mass 11.1649 -> 10.180139
- link upperArm_Link: mass 18.7946 -> 17.664060
- link wrist1_Link: mass 2.5692 -> 2.370741
- link wrist2_Link: mass 2.5692 -> 2.370741
- link wrist3_Link: mass 0.203 -> 0.259654

File: urdf/aubo_i3H.urdf (robot description, URDF)
Before this commit: robot aubo_i3H, 8 links, 7 joints
Links:
- link base_link: mass 0.97332 -> 1.365846
- link foreArm_Link: mass 1.5214 -> 2.351523
- link shoulder_Link: mass 1.173 -> 3.257300
- link upperArm_Link: mass 2.7791 -> 6.116851
- link wrist1_Link: mass 0.63348 -> 1.628022
- link wrist2_Link: mass 0.63348 -> 1.628022
- link wrist3_Link: mass 0.13713 -> 0.197800

File: urdf/aubo_i5F_34.urdf (robot description, URDF)
Before this commit: robot aubo_i5F_34, 8 links, 7 joints
Links:
- link base_link: mass 0.83419 -> 1.539020
- link foreArm_Link: mass 2.88 -> 2.849168
- link shoulder_Link: mass 5.05 -> 4.848581
- link upperArm_Link: mass 11.28 -> 10.836261
- link wrist1_Link: mass 1.62 -> 1.6280228022
- link wrist2_Link: mass 1.62 -> 1.6280228022
- link wrist3_Link: mass 0.5 -> 0.197800

File: urdf/aubo_i5H.urdf (robot description, URDF)
Before this commit: robot aubo_i5H, 8 links, 7 joints
Links:
- link base_link: mass 1.53902 -> 1.539020
- link foreArm_Link: mass 2.72848 -> 2.849168
- link shoulder_Link: mass 4.77751 -> 4.848581
- link upperArm_Link: mass 10.63494 -> 10.836261
- link wrist1_Link: mass 1.57605 -> 1.628022
- link wrist2_Link: mass 1.57605 -> 1.628022
- link wrist3_Link: mass 0.17176 -> 0.197800

File: urdf/aubo_i5_10.urdf (robot description, URDF)
Before this commit: robot aubo_i5_10, 8 links, 7 joints
Links:
- link base_link: mass 0.83419 -> 1.539020
- link foreArm_Link: mass 2.88 -> 2.849168
- link shoulder_Link: mass 5.05 -> 4.848581
- link upperArm_Link: mass 11.28 -> 10.836261
- link wrist1_Link: mass 1.62 -> 1.6280228022
- link wrist2_Link: mass 1.62 -> 1.6280228022
- link wrist3_Link: mass 0.5 -> 0.197800

File: urdf/aubo_i5_11.urdf (robot description, URDF)
Before this commit: robot aubo_i5_11, 8 links, 7 joints
Links:
- link base_link: mass 0.83419 -> 1.539020
- link foreArm_Link: mass 2.88 -> 2.849168
- link shoulder_Link: mass 5.05 -> 4.848581
- link upperArm_Link: mass 11.28 -> 10.836261
- link wrist1_Link: mass 1.62 -> 1.6280228022
- link wrist2_Link: mass 1.62 -> 1.6280228022
- link wrist3_Link: mass 0.5 -> 0.197800

File: urdf/aubo_i5_30.urdf (robot description, URDF)
Before this commit: robot aubo_i5_30, 8 links, 7 joints
Links:
- link base_link: mass 0.83419 -> 1.539020
- link foreArm_Link: mass 2.88 -> 2.849168
- link shoulder_Link: mass 5.05 -> 4.848581
- link upperArm_Link: mass 11.28 -> 10.836261
- link wrist1_Link: mass 1.62 -> 1.6280228022
- link wrist2_Link: mass 1.62 -> 1.6280228022
- link wrist3_Link: mass 0.5 -> 0.197800
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